File: forward_converter/forward_converter.sch (KiCad schematic (older format))
At the start: 31 parts

Commit message: Add files via upload
PCB design is completed except thickness and width adjustments of connections
Parts:
- removed C?: C, symbol Device:C
- removed D?: D, symbol Device:D
- removed R?: R, symbol Device:R
- removed U?: PS2801-1, symbol forward_converter_lib:PS2801-1
- added C? (x2): C, symbol Device:C
- added R?: R, symbol Device:R
Connections:
- net labels removed: GNDREF
- wire segments 91 -> 80
Changed lines of the file:
@@
 	2850 2200 2650 2200
+$Comp
+L power:GND #PWR?
+U 1 1 5EF1D190
+P 2650 2500
+F 0 "#PWR?" H 2650 2250 50  0001 C CNN
+F 1 "GND" H 2655 2327 50  0000 C CNN
+F 2 "" H 2650 2500 50  0001 C CNN
+F 3 "" H 2650 2500 50  0001 C CNN
+	1    2650 2500
+	1    0    0    -1
+$EndComp
 $Comp
 L Device:C C?
@@
 F 3 "" H 2400 2400 50  0001 C CNN
 	1    2400 2400
+	1    0    0    -1
+$EndComp
+Wire Wire Line
+	2850 2000 2200 2000
+Wire Wire Line
+	2200 2000 2200 3650
+Wire Wire Line
+	2200 3650 2850 3650
+$Comp
+L Device:R R?
+U 1 1 5EF1EE58
+P 2000 2050
+F 0 "R?" H 2070 2096 50  0000 L CNN
+F 1 "R" H 2070 2005 50  0000 L CNN
+F 2 "" V 1930 2050 50  0001 C CNN
+F 3 "~" H 2000 2050 50  0001 C CNN
+	1    2000 2050
+	1    0    0    -1
+$EndComp
+$Comp
+L Device:C C?
+U 1 1 5EF1F981
+P 2000 2450
+F 0 "C?" H 2115 2496 50  0000 L CNN
+F 1 "C" H 2115 2405 50  0000 L CNN
+F 2 "" H 2038 2300 50  0001 C CNN
+F 3 "~" H 2000 2450 50  0001 C CNN
+	1    2000 2450
+	1    0    0    -1
+$EndComp
+$Comp
+L Device:C C?
+U 1 1 5EF1FE96
+P 1700 2250
+F 0 "C?" H 1815 2296 50  0000 L CNN
+F 1 "C" H 1815 2205 50  0000 L CNN
+F 2 "" H 1738 2100 50  0001 C CNN
+F 3 "~" H 1700 2250 50  0001 C CNN
+	1    1700 2250
+	1    0    0    -1
+$EndComp
+Wire Wire Line
+	2850 1900 2000 1900
+Wire Wire Line
+	2000 1900 1700 1900
+Wire Wire Line
+	1700 1900 1700 2100
+Connection ~ 2000 1900
+Wire Wire Line
+	2000 2200 2000 2300
+$Comp
+L power:GND #PWR?
+U 1 1 5EF215D2
+P 2000 2600
+F 0 "#PWR?" H 2000 2350 50  0001 C CNN
+F 1 "GND" H 2005 2427 50  0000 C CNN
+F 2 "" H 2000 2600 50  0001 C CNN
+F 3 "" H 2000 2600 50  0001 C CNN
+	1    2000 2600
+	1    0    0    -1
+$EndComp
+$Comp
+L power:GND #PWR?
+U 1 1 5EF21BBF
+P 1700 2400
+F 0 "#PWR?" H 1700 2150 50  0001 C CNN
+F 1 "GND" H 1705 2227 50  0000 C CNN
+F 2 "" H 1700 2400 50  0001 C CNN
+F 3 "" H 1700 2400 50  0001 C CNN
+	1    1700 2400
 	1    0    0    -1
 $EndComp
@@
 	1    0    0    -1
 $EndComp
-Wire Wire Line
-	7800 1400 8200 1400
-Connection ~ 7800 1400
-Connection ~ 8200 1400
-Wire Wire Line
-	8200 1800 8200 1700
-Wire Wire Line
-	7800 1700 7800 1800
-Connection ~ 7800 1800
-Wire Wire Line
-	7800 1800 8200 1800
-Wire Wire Line
-	7050 1700 7050 1800
-Connection ~ 7050 1800
-Wire Wire Line
-	7050 1800 7800 1800
-$Comp
-L power:GND #PWR?
-U 1 1 5EF1D190
-P 2650 2500
-F 0 "#PWR?" H 2650 2250 50  0001 C CNN
-F 1 "GND" H 2655 2327 50  0000 C CNN
-F 2 "" H 2650 2500 50  0001 C CNN
-F 3 "" H 2650 2500 50  0001 C CNN
-	1    2650 2500
-	1    0    0    -1
-$EndComp
 $Comp
 L Device:R R?
@@
 	1    0    0    -1
 $EndComp
+Wire Wire Line
+	7800 1400 8200 1400
+Connection ~ 7800 1400
+Connection ~ 8200 1400
+Wire Wire Line
+	5950 1800 6350 1800
+Wire Wire Line
+	8200 1800 8200 1700
+Wire Wire Line
+	7800 1700 7800 1800
+Connection ~ 7800 1800
+Wire Wire Line
+	7800 1800 8200 1800
+Wire Wire Line
+	7050 1700 7050 1800
+Connection ~ 7050 1800
+Wire Wire Line
+	7050 1800 7800 1800
 $Comp
 L Device:C C?
@@
 Wire Wire Line
 	7700 2800 7700 3350
-Wire Wire Line
-	7700 3350 7550 3350
 Connection ~ 7700 2800
 Wire Wire Line
@@
 	8600 1700 8600 2400
 Wire Wire Line
+	8200 1400 8450 1400
+Wire Wire Line
 	8450 1400 8450 2100
-Wire Wire Line
-	8200 1400 8450 1400
+Connection ~ 8450 1400
 Wire Wire Line
 	8450 1400 8600 1400
-Connection ~ 8450 1400
 $Comp
 L Device:D_Schottky D?
@@
 Wire Wire Line
 	6350 2100 6350 1800
-Wire Wire Line
-	5950 1800 6350 1800
+Connection ~ 6350 1800
 Wire Wire Line
 	6350 1800 7050 1800
-Connection ~ 6350 1800
+Wire Wire Line
+	6350 2400 6500 2400
 Wire Wire Line
 	6500 2400 6500 3250
 Wire Wire Line
 	6500 3250 6850 3250
-Wire Wire Line
-	6350 2400 6500 2400
+Connection ~ 6500 2400
 Wire Wire Line
 	6500 2400 6700 2400
-Connection ~ 6500 2400
 $Comp
 L Device:C C?
@@
 	6500 4000 6500 3950
 Wire Wire Line
+	7700 3350 7550 3350
+Wire Wire Line
 	7550 3250 7600 3250
-$Comp
-L forward_converter_lib:PS2801-1 U?
-U 1 1 5EF58B5F
-P 5850 4400
-F 0 "U?" H 5850 4675 50  0000 C CNN
-F 1 "PS2801-1" H 5850 4584 50  0000 C CNN
-F 2 "" H 5850 4250 50  0001 C CNN
-F 3 "" H 5850 4250 50  0001 C CNN
-	1    5850 4400
-	-1   0    0    1
-$EndComp
-$Comp
-L Device:R R?
-U 1 1 5EF5E93C
-P 7600 3750
-F 0 "R?" H 7670 3796 50  0000 L CNN
-F 1 "R" H 7670 3705 50  0000 L CNN
-F 2 "" V 7530 3750 50  0001 C CNN
-F 3 "~" H 7600 3750 50  0001 C CNN
-	1    7600 3750
-	1    0    0    -1
-$EndComp
-$Comp
-L Device:D D?
-U 1 1 5EF5F720
-P 7600 4150
-F 0 "D?" V 7646 4071 50  0000 R CNN
-F 1 "D" V 7555 4071 50  0000 R CNN
-F 2 "" H 7600 4150 50  0001 C CNN
-F 3 "~" H 7600 4150 50  0001 C CNN
-	1    7600 4150
-	0    -1   -1   0
-$EndComp
-Wire Wire Line
-	7600 4450 6300 4450
-Wire Wire Line
-	7600 3250 7600 3600
-Wire Wire Line
-	7600 4300 7600 4450
-Wire Wire Line
-	7600 3900 7600 4000
-Wire Wire Line
-	6300 3600 6500 3600
-Wire Wire Line
-	6300 4100 6500 4100
-Wire Wire Line
-	6500 4100 6500 4150
-Wire Wire Line
-	6300 4350 6300 4100
-Wire Wire Line
-	6300 4100 6300 3600
-Connection ~ 6300 4100
-Wire Wire Line
-	2000 4450 2000 1900
-Wire Wire Line
-	2000 1900 2850 1900
-Wire Wire Line
-	2000 4450 5400 4450
-Wire Wire Line
-	2650 2200 2650 2000
-Wire Wire Line
-	2650 2000 2850 2000
-Connection ~ 2650 2200
-Wire Wire Line
-	5400 4350 5200 4350
-Wire Wire Line
-	5200 4350 5200 4650
-$Comp
-L power:GND #PWR?
-U 1 1 5EF79802
-P 5200 4650
-F 0 "#PWR?" H 5200 4400 50  0001 C CNN
-F 1 "GND" H 5205 4477 50  0000 C CNN
-F 2 "" H 5200 4650 50  0001 C CNN
-F 3 "" H 5200 4650 50  0001 C CNN
-	1    5200 4650
-	1    0    0    -1
-$EndComp
-Wire Wire Line
-	3350 2100 3350 2700
-$Comp
-L power:GND #PWR?
-U 1 1 5EF7E95F
-P 3350 2700
-F 0 "#PWR?" H 3350 2450 50  0001 C CNN
-F 1 "GND" H 3355 2527 50  0000 C CNN
-F 2 "" H 3350 2700 50  0001 C CNN
-F 3 "" H 3350 2700 50  0001 C CNN
-	1    3350 2700
-	1    0    0    -1
-$EndComp
-$Comp
-L power:GNDREF #PWR?
-U 1 1 5EF7F262
-P 6500 4150
-F 0 "#PWR?" H 6500 3900 50  0001 C CNN
-F 1 "GNDREF" H 6505 3977 50  0000 C CNN
-F 2 "" H 6500 4150 50  0001 C CNN
-F 3 "" H 6500 4150 50  0001 C CNN
-	1    6500 4150
-	1    0    0    -1
-$EndComp
-$Comp
-L power:GNDREF #PWR?
-U 1 1 5EF7F88A
-P 8600 3150
-F 0 "#PWR?" H 8600 2900 50  0001 C CNN
-F 1 "GNDREF" H 8605 2977 50  0000 C CNN
-F 2 "" H 8600 3150 50  0001 C CNN
-F 3 "" H 8600 3150 50  0001 C CNN
-	1    8600 3150
-	1    0    0    -1
-$EndComp
-$Comp
-L Device:C C?
-U 1 1 5EF803A6
-P 5850 4100
-F 0 "C?" V 5598 4100 50  0000 C CNN
-F 1 "C" V 5689 4100 50  0000 C CNN
-F 2 "" H 5888 3950 50  0001 C CNN
-F 3 "~" H 5850 4100 50  0001 C CNN
-	1    5850 4100
-	0    1    1    0
-$EndComp
-Wire Wire Line
-	6000 4100 6300 4100
-Wire Wire Line
-	5700 4100 5200 4100
-Wire Wire Line
-	5200 4100 5200 4350
-Connection ~ 5200 4350
+Wire Wire Line
+	7600 3250 7600 4200
+Wire Wire Line
+	7600 4200 7050 4200
 $EndSCHEMATC

Commit message: Controller calculations completed and new mosfet selected
Parts:
- removed C? (x2): C, symbol Device:C
- removed R?: R, symbol Device:R
- added C?: C, symbol Device:C
- added D?: D, symbol Device:D
- added R?: R, symbol Device:R
- added U?: PS2801-1, symbol forward_converter_lib:PS2801-1
Connections:
- net labels added: GNDREF
- wire segments 80 -> 91
Changed lines of the file:
@@
 	2850 2200 2650 2200
-$Comp
-L power:GND #PWR?
-U 1 1 5EF1D190
-P 2650 2500
-F 0 "#PWR?" H 2650 2250 50  0001 C CNN
-F 1 "GND" H 2655 2327 50  0000 C CNN
-F 2 "" H 2650 2500 50  0001 C CNN
-F 3 "" H 2650 2500 50  0001 C CNN
-	1    2650 2500
-	1    0    0    -1
-$EndComp
 $Comp
 L Device:C C?
@@
 F 3 "" H 2400 2400 50  0001 C CNN
 	1    2400 2400
-	1    0    0    -1
-$EndComp
-Wire Wire Line
-	2850 2000 2200 2000
-Wire Wire Line
-	2200 2000 2200 3650
-Wire Wire Line
-	2200 3650 2850 3650
-$Comp
-L Device:R R?
-U 1 1 5EF1EE58
-P 2000 2050
-F 0 "R?" H 2070 2096 50  0000 L CNN
-F 1 "R" H 2070 2005 50  0000 L CNN
-F 2 "" V 1930 2050 50  0001 C CNN
-F 3 "~" H 2000 2050 50  0001 C CNN
-	1    2000 2050
-	1    0    0    -1
-$EndComp
-$Comp
-L Device:C C?
-U 1 1 5EF1F981
-P 2000 2450
-F 0 "C?" H 2115 2496 50  0000 L CNN
-F 1 "C" H 2115 2405 50  0000 L CNN
-F 2 "" H 2038 2300 50  0001 C CNN
-F 3 "~" H 2000 2450 50  0001 C CNN
-	1    2000 2450
-	1    0    0    -1
-$EndComp
-$Comp
-L Device:C C?
-U 1 1 5EF1FE96
-P 1700 2250
-F 0 "C?" H 1815 2296 50  0000 L CNN
-F 1 "C" H 1815 2205 50  0000 L CNN
-F 2 "" H 1738 2100 50  0001 C CNN
-F 3 "~" H 1700 2250 50  0001 C CNN
-	1    1700 2250
-	1    0    0    -1
-$EndComp
-Wire Wire Line
-	2850 1900 2000 1900
-Wire Wire Line
-	2000 1900 1700 1900
-Wire Wire Line
-	1700 1900 1700 2100
-Connection ~ 2000 1900
-Wire Wire Line
-	2000 2200 2000 2300
-$Comp
-L power:GND #PWR?
-U 1 1 5EF215D2
-P 2000 2600
-F 0 "#PWR?" H 2000 2350 50  0001 C CNN
-F 1 "GND" H 2005 2427 50  0000 C CNN
-F 2 "" H 2000 2600 50  0001 C CNN
-F 3 "" H 2000 2600 50  0001 C CNN
-	1    2000 2600
-	1    0    0    -1
-$EndComp
-$Comp
-L power:GND #PWR?
-U 1 1 5EF21BBF
-P 1700 2400
-F 0 "#PWR?" H 1700 2150 50  0001 C CNN
-F 1 "GND" H 1705 2227 50  0000 C CNN
-F 2 "" H 1700 2400 50  0001 C CNN
-F 3 "" H 1700 2400 50  0001 C CNN
-	1    1700 2400
 	1    0    0    -1
 $EndComp
@@
 	1    0    0    -1
 $EndComp
+Wire Wire Line
+	7800 1400 8200 1400
+Connection ~ 7800 1400
+Connection ~ 8200 1400
+Wire Wire Line
+	8200 1800 8200 1700
+Wire Wire Line
+	7800 1700 7800 1800
+Connection ~ 7800 1800
+Wire Wire Line
+	7800 1800 8200 1800
+Wire Wire Line
+	7050 1700 7050 1800
+Connection ~ 7050 1800
+Wire Wire Line
+	7050 1800 7800 1800
+$Comp
+L power:GND #PWR?
+U 1 1 5EF1D190
+P 2650 2500
+F 0 "#PWR?" H 2650 2250 50  0001 C CNN
+F 1 "GND" H 2655 2327 50  0000 C CNN
+F 2 "" H 2650 2500 50  0001 C CNN
+F 3 "" H 2650 2500 50  0001 C CNN
+	1    2650 2500
+	1    0    0    -1
+$EndComp
 $Comp
 L Device:R R?
@@
 	1    0    0    -1
 $EndComp
-Wire Wire Line
-	7800 1400 8200 1400
-Connection ~ 7800 1400
-Connection ~ 8200 1400
-Wire Wire Line
-	5950 1800 6350 1800
-Wire Wire Line
-	8200 1800 8200 1700
-Wire Wire Line
-	7800 1700 7800 1800
-Connection ~ 7800 1800
-Wire Wire Line
-	7800 1800 8200 1800
-Wire Wire Line
-	7050 1700 7050 1800
-Connection ~ 7050 1800
-Wire Wire Line
-	7050 1800 7800 1800
 $Comp
 L Device:C C?
@@
 Wire Wire Line
 	7700 2800 7700 3350
+Wire Wire Line
+	7700 3350 7550 3350
 Connection ~ 7700 2800
 Wire Wire Line
@@
 	8600 1700 8600 2400
 Wire Wire Line
+	8450 1400 8450 2100
+Wire Wire Line
 	8200 1400 8450 1400
 Wire Wire Line
-	8450 1400 8450 2100
+	8450 1400 8600 1400
 Connection ~ 8450 1400
-Wire Wire Line
-	8450 1400 8600 1400
 $Comp
 L Device:D_Schottky D?
@@
 Wire Wire Line
 	6350 2100 6350 1800
+Wire Wire Line
+	5950 1800 6350 1800
+Wire Wire Line
+	6350 1800 7050 1800
 Connection ~ 6350 1800
 Wire Wire Line
-	6350 1800 7050 1800
+	6500 2400 6500 3250
+Wire Wire Line
+	6500 3250 6850 3250
 Wire Wire Line
 	6350 2400 6500 2400
 Wire Wire Line
-	6500 2400 6500 3250
-Wire Wire Line
-	6500 3250 6850 3250
+	6500 2400 6700 2400
 Connection ~ 6500 2400
-Wire Wire Line
-	6500 2400 6700 2400
 $Comp
 L Device:C C?
@@
 	6500 4000 6500 3950
 Wire Wire Line
-	7700 3350 7550 3350
-Wire Wire Line
 	7550 3250 7600 3250
-Wire Wire Line
-	7600 3250 7600 4200
-Wire Wire Line
-	7600 4200 7050 4200
+$Comp
+L forward_converter_lib:PS2801-1 U?
+U 1 1 5EF58B5F
+P 5850 4400
+F 0 "U?" H 5850 4675 50  0000 C CNN
+F 1 "PS2801-1" H 5850 4584 50  0000 C CNN
+F 2 "" H 5850 4250 50  0001 C CNN
+F 3 "" H 5850 4250 50  0001 C CNN
+	1    5850 4400
+	-1   0    0    1
+$EndComp
+$Comp
+L Device:R R?
+U 1 1 5EF5E93C
+P 7600 3750
+F 0 "R?" H 7670 3796 50  0000 L CNN
+F 1 "R" H 7670 3705 50  0000 L CNN
+F 2 "" V 7530 3750 50  0001 C CNN
+F 3 "~" H 7600 3750 50  0001 C CNN
+	1    7600 3750
+	1    0    0    -1
+$EndComp
+$Comp
+L Device:D D?
+U 1 1 5EF5F720
+P 7600 4150
+F 0 "D?" V 7646 4071 50  0000 R CNN
+F 1 "D" V 7555 4071 50  0000 R CNN
+F 2 "" H 7600 4150 50  0001 C CNN
+F 3 "~" H 7600 4150 50  0001 C CNN
+	1    7600 4150
+	0    -1   -1   0
+$EndComp
+Wire Wire Line
+	7600 4450 6300 4450
+Wire Wire Line
+	7600 3250 7600 3600
+Wire Wire Line
+	7600 4300 7600 4450
+Wire Wire Line
+	7600 3900 7600 4000
+Wire Wire Line
+	6300 3600 6500 3600
+Wire Wire Line
+	6300 4100 6500 4100
+Wire Wire Line
+	6500 4100 6500 4150
+Wire Wire Line
+	6300 4350 6300 4100
+Wire Wire Line
+	6300 4100 6300 3600
+Connection ~ 6300 4100
+Wire Wire Line
+	2000 4450 2000 1900
+Wire Wire Line
+	2000 1900 2850 1900
+Wire Wire Line
+	2000 4450 5400 4450
+Wire Wire Line
+	2650 2200 2650 2000
+Wire Wire Line
+	2650 2000 2850 2000
+Connection ~ 2650 2200
+Wire Wire Line
+	5400 4350 5200 4350
+Wire Wire Line
+	5200 4350 5200 4650
+$Comp
+L power:GND #PWR?
+U 1 1 5EF79802
+P 5200 4650
+F 0 "#PWR?" H 5200 4400 50  0001 C CNN
+F 1 "GND" H 5205 4477 50  0000 C CNN
+F 2 "" H 5200 4650 50  0001 C CNN
+F 3 "" H 5200 4650 50  0001 C CNN
+	1    5200 4650
+	1    0    0    -1
+$EndComp
+Wire Wire Line
+	3350 2100 3350 2700
+$Comp
+L power:GND #PWR?
+U 1 1 5EF7E95F
+P 3350 2700
+F 0 "#PWR?" H 3350 2450 50  0001 C CNN
+F 1 "GND" H 3355 2527 50  0000 C CNN
+F 2 "" H 3350 2700 50  0001 C CNN
+F 3 "" H 3350 2700 50  0001 C CNN
+	1    3350 2700
+	1    0    0    -1
+$EndComp
+$Comp
+L power:GNDREF #PWR?
+U 1 1 5EF7F262
+P 6500 4150
+F 0 "#PWR?" H 6500 3900 50  0001 C CNN
+F 1 "GNDREF" H 6505 3977 50  0000 C CNN
+F 2 "" H 6500 4150 50  0001 C CNN
+F 3 "" H 6500 4150 50  0001 C CNN
+	1    6500 4150
+	1    0    0    -1
+$EndComp
+$Comp
+L power:GNDREF #PWR?
+U 1 1 5EF7F88A
+P 8600 3150
+F 0 "#PWR?" H 8600 2900 50  0001 C CNN
+F 1 "GNDREF" H 8605 2977 50  0000 C CNN
+F 2 "" H 8600 3150 50  0001 C CNN
+F 3 "" H 8600 3150 50  0001 C CNN
+	1    8600 3150
+	1    0    0    -1
+$EndComp
+$Comp
+L Device:C C?
+U 1 1 5EF803A6
+P 5850 4100
+F 0 "C?" V 5598 4100 50  0000 C CNN
+F 1 "C" V 5689 4100 50  0000 C CNN
+F 2 "" H 5888 3950 50  0001 C CNN
+F 3 "~" H 5850 4100 50  0001 C CNN
+	1    5850 4100
+	0    1    1    0
+$EndComp
+Wire Wire Line
+	6000 4100 6300 4100
+Wire Wire Line
+	5700 4100 5200 4100
+Wire Wire Line
+	5200 4100 5200 4350
+Connection ~ 5200 4350
 $EndSCHEMATC
