File: forward_converter/_autosave-forward_converter_opto.kicad_pcb (KiCad board)
At the start: 2 copper layers, 302.3 x 137.2 mm, 23 parts, among them J1 Conn_Coaxial, J2 Conn_Coaxial, J3 Conn_Coaxial, J4 Conn_Coaxial, Q1 IRF740, U1 LT3758, U2 designed_transformer_model

Commit message: Add files via upload
PCB design is completed except thickness and width adjustments of connections
Parts:
- moved J4 47.8 mm to (171.4, 96.5), turned to 270 degrees
- moved J3 29.7 mm to (210.8, 96.5), turned to 270 degrees
Routing:
- net GNDA: track 230.3 -> 188.2 mm
- net Net-(C5-Pad1): track 97.0 -> 111.2 mm
