File: forward_converter/_autosave-forward_converter_opto.kicad_pcb (KiCad board)
At the start: 2 copper layers, 302.3 x 111.8 mm, 23 parts, among them J1 Conn_Coaxial, J2 Conn_Coaxial, J3 Conn_Coaxial, J4 Conn_Coaxial, Q1 IRF740, U1 LT3758, U2 designed_transformer_model

Commit message: Add files via upload
Routing:
- removed copper zone on B.Cu, net GND
- removed copper zone on B.Cu, net GNDA
Changed lines of the file:
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@@
   (segment (start 25.74 61.3) (end 47.92 61.3) (width 0.4) (layer F.Cu) (net 18))
   (segment (start -8.89 26.67) (end 25.74 61.3) (width 0.4) (layer F.Cu) (net 18))
-  (zone (net 6) (net_name GNDA) (layer B.Cu) (hatch edge 0.508)
-    (connect_pads (clearance 0.508))
-    (min_thickness 0.254)
-    (fill yes (arc_segments 32) (thermal_gap 0.508) (thermal_bridge_width 0.508))
-    (polygon
-      (pts
-        (xy 274.32 102.87) (xy 138.43 102.87) (xy 138.43 19.05) (xy 274.32 19.05)
-      )
-    )
-  )
-  (zone (net 1) (net_name GND) (layer B.Cu) (hatch edge 0.508)
-    (connect_pads (clearance 0.508))
-    (min_thickness 0.254)
-    (fill yes (arc_segments 32) (thermal_gap 0.508) (thermal_bridge_width 0.508))
-    (polygon
-      (pts
-        (xy 95.25 121.92) (xy -21.59 121.92) (xy -21.59 53.34) (xy 95.25 53.34)
-      )
-    )
-  )
 )
